File: domino.kicad_pcb (KiCad board)
At the start: 2 copper layers, 190.5 x 57.2 mm, 69 parts, among them SW1 SW_PUSH, U1 ProMicro

Commit message: uhhh
Changed lines of the file:
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@@
     (add_net "Net-(U1-Pad9)")
+  )
+  (module rainstuff:tht-reset (layer F.Cu)
+    (at 74.6125 15.08125)
+    (fp_text reference SW1 (at 0 0.5 180) (layer F.SilkS) hide
+      (effects (font (size 1 1) (thickness 0.15)))
+    )
+    (fp_text value SW_PUSH (at 0 -0.5 180) (layer F.Fab)
+      (effects (font (size 1 1) (thickness 0.15)))
+    )
+    (fp_line (start 3 -1) (end -3 -1) (layer F.SilkS) (width 0.12))
+    (fp_line (start 3 1) (end 3 -1) (layer F.SilkS) (width 0.12))
+    (fp_line (start -3 1) (end 3 1) (layer F.SilkS) (width 0.12))
+    (fp_line (start -3 -1) (end -3 1) (layer F.SilkS) (width 0.12))
+    (fp_line (start 3 -1) (end -3 -1) (layer B.SilkS) (width 0.12))
+    (fp_line (start 3 1) (end 3 -1) (layer B.SilkS) (width 0.12))
+    (fp_line (start -3 1) (end 3 1) (layer B.SilkS) (width 0.12))
+    (fp_line (start -3 -1) (end -3 1) (layer B.SilkS) (width 0.12))
+    (pad 2 thru_hole oval (at 3 0) (size 1.524 3) (drill oval 0.762 2) (layers *.Cu *.Mask)
+      (net 30 "Net-(SW1-Pad2)"))
+    (pad 1 thru_hole oval (at -3 0) (size 1.524 3) (drill oval 0.762 2) (layers *.Cu *.Mask)
+      (net 51 GND))
   )
   (module Diode_THT:D_DO-35_SOD27_P7.62mm_Horizontal (layer B.Cu)
@@
     (pad "" np_thru_hole circle (at 11.90625 -8.255) (size 3.9878 3.9878) (drill 3.9878) (layers *.Cu *.Mask))
   )
-  (module rainstuff:tht-reset (layer F.Cu)
-    (at 74.6125 15.08125)
-    (fp_text reference SW1 (at 0 0.5 180) (layer F.SilkS) hide
-      (effects (font (size 1 1) (thickness 0.15)))
-    )
-    (fp_text value SW_PUSH (at 0 -0.5 180) (layer F.Fab)
-      (effects (font (size 1 1) (thickness 0.15)))
-    )
-    (fp_line (start 3 -1) (end -3 -1) (layer F.SilkS) (width 0.12))
-    (fp_line (start 3 1) (end 3 -1) (layer F.SilkS) (width 0.12))
-    (fp_line (start -3 1) (end 3 1) (layer F.SilkS) (width 0.12))
-    (fp_line (start -3 -1) (end -3 1) (layer F.SilkS) (width 0.12))
-    (fp_line (start 3 -1) (end -3 -1) (layer B.SilkS) (width 0.12))
-    (fp_line (start 3 1) (end 3 -1) (layer B.SilkS) (width 0.12))
-    (fp_line (start -3 1) (end 3 1) (layer B.SilkS) (width 0.12))
-    (fp_line (start -3 -1) (end -3 1) (layer B.SilkS) (width 0.12))
-    (pad 2 thru_hole circle (at 3 0) (size 1.524 1.524) (drill 0.762) (layers *.Cu *.Mask)
-      (net 30 "Net-(SW1-Pad2)"))
-    (pad 1 thru_hole circle (at -3 0) (size 1.524 1.524) (drill 0.762) (layers *.Cu *.Mask)
-      (net 51 GND))
-  )
   (module MX_Only:MXOnly-1U-NoLED (layer F.Cu)
